File: mothbeam12V.kicad_sch (KiCad schematic)
At the start: 25 parts, among them J1 +VDC, J3 EN, J8 GND, SW2 SW_DIP_x04, U1 BCR420U, U2 BCR420U, U3 BCR420U

Commit message: added OSHWA license, pdf and schematics
Other:
- note added: "Certified as open source hardware by the Open Source Hardware Association"
- note added: "Designed by LabLab http://www.lablab.eu"
- note added: "USE IMS (insulated metal substrate) PCB material"
